File: pcb/motor_controllers/MC_board.sch (KiCad schematic (older format))
At the start: 31 parts, among them J12V1 Screw_Terminal_01x02, J12V2 Screw_Terminal_01x02, J12V3 Screw_Terminal_01x02, J12V4 Screw_Terminal_01x02, J2 RJ45, J5V1 Screw_Terminal_01x02, J5V2 Screw_Terminal_01x02, J9V1 Screw_Terminal_01x02, U1 Teensy3.2, U2 MAX98306

Commit message: Added rules
Parts:
- added JP1: gnd jumper, symbol Jumper:Jumper_2_Open
Connections:
- net GND: now also JP1.1 (A)
- net GND1: now also JP1.2 (B)
Changed lines of the file:
@@
 	1    0    0    -1
 $EndComp
+$Comp
+L Jumper:Jumper_2_Open JP1
+U 1 1 5F0D8BE7
+P 3600 13100
+F 0 "JP1" H 3600 13335 50  0000 C CNN
+F 1 "gnd jumper" H 3600 13244 50  0000 C CNN
+F 2 "" H 3600 13100 50  0001 C CNN
+F 3 "~" H 3600 13100 50  0001 C CNN
+	1    3600 13100
+	1    0    0    -1
+$EndComp
+Wire Wire Line
+	2650 14150 2700 14150
+Wire Wire Line
+	3400 14150 3400 13100
+Connection ~ 2700 14150
+Wire Wire Line
+	2700 14150 3400 14150
+Wire Wire Line
+	2650 13450 2700 13450
+Wire Wire Line
+	3800 13450 3800 13100
+Connection ~ 2700 13450
+Wire Wire Line
+	2700 13450 3800 13450
 $EndSCHEMATC

Commit message: Flipped motor controller for space, added switches
Parts:
- added SW12: SW12V, Button_Switch_THT:SW_DIP_SPSTx01_Piano_10.8x4.1mm_W7.62mm_P2.54mm, symbol Switch:SW_SPST
- added SW5: SW5V, Button_Switch_THT:SW_DIP_SPSTx01_Piano_10.8x4.1mm_W7.62mm_P2.54mm, symbol Switch:SW_SPST
- added SW9: SW9V, Button_Switch_THT:SW_DIP_SPSTx01_Piano_10.8x4.1mm_W7.62mm_P2.54mm, symbol Switch:SW_SPST
Connections:
- net +12V: now also SW12.2 (B); no longer 12V1.1
- net +5V: now also SW5.2 (B); no longer 5V1.1
- net +9V: now also SW9.2 (B); no longer 9V1.1
- net GND: now also JP1.2 (B); no longer JP1.1 (A)
- net GND1: now also JP1.1 (A); no longer JP1.2 (B)
- new net: 9V1.1, SW9.1 (A)
- new net: 5V1.1, SW5.1 (A)
- new net: 12V1.1, SW12.1 (A)
Other:
- moved on the sheet: JP1
Changed lines of the file:
@@
-$EndComp
-$Comp
-L Connector:Barrel_Jack 5V1
-U 1 1 5F03C8F5
-P 2400 14050
-F 0 "5V1" H 2457 14375 50  0000 C CNN
-F 1 "5V" H 2457 14284 50  0000 C CNN
-F 2 "Connector_BarrelJack:BarrelJack_Horizontal" H 2450 14010 50  0001 C CNN
-F 3 "~" H 2450 14010 50  0001 C CNN
-	1    2400 14050
-	1    0    0    -1
 $EndComp
 $Comp
@@
 L power:+9V #PWR0122
 U 1 1 5F366504
-P 2700 13250
-F 0 "#PWR0122" H 2700 13100 50  0001 C CNN
-F 1 "+9V" H 2715 13423 50  0000 C CNN
-F 2 "" H 2700 13250 50  0001 C CNN
-F 3 "" H 2700 13250 50  0001 C CNN
-	1    2700 13250
-	1    0    0    -1
+P 3100 13250
+F 0 "#PWR0122" H 3100 13100 50  0001 C CNN
+F 1 "+9V" H 3115 13423 50  0000 C CNN
+F 2 "" H 3100 13250 50  0001 C CNN
+F 3 "" H 3100 13250 50  0001 C CNN
+	1    3100 13250
+	0    1    1    0
 $EndComp
 $Comp
@@
 L power:+12V #PWR0135
 U 1 1 5F240265
-P 2700 12450
-F 0 "#PWR0135" H 2700 12300 50  0001 C CNN
-F 1 "+12V" H 2715 12623 50  0000 C CNN
-F 2 "" H 2700 12450 50  0001 C CNN
-F 3 "" H 2700 12450 50  0001 C CNN
-	1    2700 12450
-	1    0    0    -1
+P 3100 12450
+F 0 "#PWR0135" H 3100 12300 50  0001 C CNN
+F 1 "+12V" H 3115 12623 50  0000 C CNN
+F 2 "" H 3100 12450 50  0001 C CNN
+F 3 "" H 3100 12450 50  0001 C CNN
+	1    3100 12450
+	0    1    1    0
 $EndComp
 $Comp
@@
 L power:+5V #PWR0137
 U 1 1 5F27D89B
-P 2700 13950
-F 0 "#PWR0137" H 2700 13800 50  0001 C CNN
-F 1 "+5V" H 2715 14123 50  0000 C CNN
-F 2 "" H 2700 13950 50  0001 C CNN
-F 3 "" H 2700 13950 50  0001 C CNN
-	1    2700 13950
-	1    0    0    -1
+P 3100 13950
+F 0 "#PWR0137" H 3100 13800 50  0001 C CNN
+F 1 "+5V" H 3115 14123 50  0000 C CNN
+F 2 "" H 3100 13950 50  0001 C CNN
+F 3 "" H 3100 13950 50  0001 C CNN
+	1    3100 13950
+	0    1    1    0
 $EndComp
 $Comp
@@
 L Jumper:Jumper_2_Open JP1
 U 1 1 5F0D8BE7
-P 3600 13100
-F 0 "JP1" H 3600 13335 50  0000 C CNN
-F 1 "gnd jumper" H 3600 13244 50  0000 C CNN
-F 2 "" H 3600 13100 50  0001 C CNN
-F 3 "~" H 3600 13100 50  0001 C CNN
-	1    3600 13100
-	1    0    0    -1
-$EndComp
-Wire Wire Line
-	2650 14150 2700 14150
-Wire Wire Line
-	3400 14150 3400 13100
+P 3550 13750
+F 0 "JP1" H 3550 13985 50  0000 C CNN
+F 1 "gnd jumper" H 3550 13894 50  0000 C CNN
+F 2 "" H 3550 13750 50  0001 C CNN
+F 3 "~" H 3550 13750 50  0001 C CNN
+	1    3550 13750
+	0    1    1    0
+$EndComp
+Wire Wire Line
+	3550 13450 3550 13550
+Wire Wire Line
+	2700 13450 3550 13450
+Connection ~ 2700 13450
+Wire Wire Line
+	2700 14150 3550 14150
+Wire Wire Line
+	3550 14150 3550 13950
 Connection ~ 2700 14150
-Wire Wire Line
-	2700 14150 3400 14150
-Wire Wire Line
-	2650 13450 2700 13450
-Wire Wire Line
-	3800 13450 3800 13100
-Connection ~ 2700 13450
-Wire Wire Line
-	2700 13450 3800 13450
+$Comp
+L Switch:SW_SPST SW12
+U 1 1 5F1753A3
+P 2900 12450
+F 0 "SW12" H 2900 12685 50  0000 C CNN
+F 1 "SW12V" H 2900 12594 50  0000 C CNN
+F 2 "Button_Switch_THT:SW_DIP_SPSTx01_Piano_10.8x4.1mm_W7.62mm_P2.54mm" H 2900 12450 50  0001 C CNN
+F 3 "~" H 2900 12450 50  0001 C CNN
+	1    2900 12450
+	1    0    0    -1
+$EndComp
+$Comp
+L Switch:SW_SPST SW9
+U 1 1 5F1934EC
+P 2900 13250
+F 0 "SW9" H 2900 13485 50  0000 C CNN
+F 1 "SW9V" H 2900 13394 50  0000 C CNN
+F 2 "Button_Switch_THT:SW_DIP_SPSTx01_Piano_10.8x4.1mm_W7.62mm_P2.54mm" H 2900 13250 50  0001 C CNN
+F 3 "~" H 2900 13250 50  0001 C CNN
+	1    2900 13250
+	1    0    0    -1
+$EndComp
+$Comp
+L Connector:Barrel_Jack 5V1
+U 1 1 5F03C8F5
+P 2400 14050
+F 0 "5V1" H 2457 14375 50  0000 C CNN
+F 1 "5V" H 2457 14284 50  0000 C CNN
+F 2 "Connector_BarrelJack:BarrelJack_Horizontal" H 2450 14010 50  0001 C CNN
+F 3 "~" H 2450 14010 50  0001 C CNN
+	1    2400 14050
+	1    0    0    -1
+$EndComp
+$Comp
+L Switch:SW_SPST SW5
+U 1 1 5F1BBE09
+P 2900 13950
+F 0 "SW5" H 2900 14185 50  0000 C CNN
+F 1 "SW5V" H 2900 14094 50  0000 C CNN
+F 2 "Button_Switch_THT:SW_DIP_SPSTx01_Piano_10.8x4.1mm_W7.62mm_P2.54mm" H 2900 13950 50  0001 C CNN
+F 3 "~" H 2900 13950 50  0001 C CNN
+	1    2900 13950
+	1    0    0    -1
+$EndComp
 $EndSCHEMATC

Commit message: Added switch footprint. Updated wiring.
Parts:
- JP1: footprint (none) -> Jumper:SolderJumper-2_P1.3mm_Open_Pad1.0x1.5mm
- SW12, SW5, SW9: footprint Button_Switch_THT:SW_DIP_SPSTx01_Piano_10.8x4.1mm_W7.62mm_P2.54mm -> teensy:SW_L102021ML04Q
Changed lines of the file:
@@
 F 0 "JP1" H 3550 13985 50  0000 C CNN
 F 1 "gnd jumper" H 3550 13894 50  0000 C CNN
-F 2 "" H 3550 13750 50  0001 C CNN
+F 2 "Jumper:SolderJumper-2_P1.3mm_Open_Pad1.0x1.5mm" H 3550 13750 50  0001 C CNN
 F 3 "~" H 3550 13750 50  0001 C CNN
 	1    3550 13750
@@
 F 0 "SW12" H 2900 12685 50  0000 C CNN
 F 1 "SW12V" H 2900 12594 50  0000 C CNN
-F 2 "Button_Switch_THT:SW_DIP_SPSTx01_Piano_10.8x4.1mm_W7.62mm_P2.54mm" H 2900 12450 50  0001 C CNN
+F 2 "teensy:SW_L102021ML04Q" H 2900 12450 50  0001 C CNN
 F 3 "~" H 2900 12450 50  0001 C CNN
 	1    2900 12450
@@
 F 0 "SW9" H 2900 13485 50  0000 C CNN
 F 1 "SW9V" H 2900 13394 50  0000 C CNN
-F 2 "Button_Switch_THT:SW_DIP_SPSTx01_Piano_10.8x4.1mm_W7.62mm_P2.54mm" H 2900 13250 50  0001 C CNN
+F 2 "teensy:SW_L102021ML04Q" H 2900 13250 50  0001 C CNN
 F 3 "~" H 2900 13250 50  0001 C CNN
 	1    2900 13250
@@
 F 0 "SW5" H 2900 14185 50  0000 C CNN
 F 1 "SW5V" H 2900 14094 50  0000 C CNN
-F 2 "Button_Switch_THT:SW_DIP_SPSTx01_Piano_10.8x4.1mm_W7.62mm_P2.54mm" H 2900 13950 50  0001 C CNN
+F 2 "teensy:SW_L102021ML04Q" H 2900 13950 50  0001 C CNN
 F 3 "~" H 2900 13950 50  0001 C CNN
 	1    2900 13950
