File: pcb/controller/MC_board.kicad_pcb (KiCad board)
At the start: 2 copper layers, 151.1 x 123.2 mm, 38 parts, among them J12V1 Screw_Terminal_01x02, J12V2 Screw_Terminal_01x02, J12V3 Screw_Terminal_01x02, J12V4 Screw_Terminal_01x02, J2 RJ45, J5V1 Screw_Terminal_01x02, J5V2 Screw_Terminal_01x02, J9V1 Screw_Terminal_01x02, SW12 SW12V, SW5 SW5V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

Commit message: renamed motor controller. Cleaning up.
Routing:
- net GND1: track 217.6 -> 209.4 mm
Other:
- board text added: "1. spout lick 2. audio + 3. audio - 4. motor zero 5. ground 6. visual stim"
- board text added: "1. touch 2. actuator + 3. actuator - 4. motor zero 5. ground"
- board text added: "Analog 1. GND 2. left audio 3. right audio 4. left visual 5. right visual 6. left actuator 7. right actuator 8. distractor"
