File: pcb/controller/controller.kicad_pcb (KiCad board)
At the start: 2 copper layers, 151.1 x 123.2 mm, 38 parts, among them J12V1 Screw_Terminal_01x02, J12V2 Screw_Terminal_01x02, J12V3 Screw_Terminal_01x02, J12V4 Screw_Terminal_01x02, J2 RJ45, J5V1 Screw_Terminal_01x02, J5V2 Screw_Terminal_01x02, J9V1 Screw_Terminal_01x02, SW12 SW12V, SW5 SW5V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

Commit message: Controller pcb working version.
Parts:
- G***: footprint teensey:churchland_lab_logo -> teensy:churchland_lab_logo
- HandleL-ToMotor1, HandleR-ToMotor1, SpoutL-ToMotor1, SpoutR-ToMotor1: footprint teensey:TerminalBlock_TE_282825-4_1x04_P5.08mm_Horizontal -> teensy:TerminalBlock_TE_282825-4_1x04_P5.08mm_Horizontal
- J12V1, J12V2, J12V3, J12V4, J5V1, J5V2, J9V1, distractor1: footprint teensey:TerminalBlock_TE_282825-2_1x02_P5.08mm_Horizontal -> teensy:TerminalBlock_TE_282825-2_1x02_P5.08mm_Horizontal
- J2: footprint teensey:RJ45_sparkfun -> teensy:RJ45_sparkfun
- JP1: footprint TestPoint:TestPoint_Bridge_Pitch2.54mm_Drill1.0mm -> TestPoint:TestPoint_2Pads_Pitch5.08mm_Drill1.3mm
- SoundVisionL1, SoundVisionR1: footprint teensey:TerminalBlock_TE_282825-6_1x06_P5.08mm_Horizontal -> teensy:TerminalBlock_TE_282825-6_1x06_P5.08mm_Horizontal
- ToHandleL1, ToHandleR1, sync_trigger_out1: footprint teensey:TerminalBlock_TE_282825-5_1x05_P5.08mm_Horizontal -> teensy:TerminalBlock_TE_282825-5_1x05_P5.08mm_Horizontal
- U1: footprint teensey:Teensy30_31_32_LC -> teensy:Teensy30_31_32_LC
- mount1, mount2: value MountingHole_6.5mm_Pad -> MountingHole_3.2mm_M3_Pad; footprint MountingHole:MountingHole_6.5mm_Pad -> MountingHole:MountingHole_3.2mm_M3_Pad
- moved SpoutR-ToMotor1 179.0 mm to (227.3, 85.1), turned to 270 degrees
- moved SpoutL-ToMotor1 171.4 mm to (185.4, 85.1), turned to 270 degrees
- moved MC-LeverR1 169.8 mm to (203.2, 33.0), turned to 0 degrees
- moved HandleR-ToMotor1 163.0 mm to (207.0, 85.1), turned to 270 degrees
- moved HandleL-ToMotor1 155.6 mm to (165.1, 85.1), turned to 270 degrees
- moved MC-SpoutR1 147.4 mm to (203.2, 58.4), turned to 0 degrees
- moved MC-LeverL1 124.6 mm to (175.3, 33.0), turned to 0 degrees
- moved C1 119.8 mm to (195.6, 74.9)
- moved J9V1 110.4 mm to (231.1, 36.8)
- moved C3 109.6 mm to (195.6, 49.5)
- moved SW9 108.2 mm to (227.3, 76.2)
- moved 9V1 108.2 mm to (226.1, 49.5)
- moved C2 96.6 mm to (167.6, 49.5)
- moved MC-SpoutL1 91.7 mm to (175.3, 58.4), turned to 0 degrees
- moved mount2 89.1 mm to (143.5, 76.2)
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Routing:
- net GND: track 69.5 -> 577.3 mm, vias 0 -> 1
- net +5V: track 151.8 -> 324.8 mm, vias 2 -> 3
- net Net-(MC-LeverR1-Pad16): track 81.5 -> 215.3 mm, vias 2 -> 1
- net +12V: track 154.0 -> 64.6 mm
- net Net-(MC-SpoutL1-Pad6): track 116.9 -> 33.4 mm
- net Net-(MC-SpoutL1-Pad5): track 108.5 -> 30.9 mm
- net Net-(MC-SpoutL1-Pad4): track 91.6 -> 23.3 mm, vias 1 -> 0
- net Net-(MC-SpoutL1-Pad3): track 98.4 -> 32.9 mm
- net Net-(MC-LeverR1-Pad15): track 82.5 -> 136.3 mm, vias 0 -> 1
- net Net-(HandleL-ToMotor1-Pad4): track 113.0 -> 64.4 mm, vias 0 -> 1
- net Net-(MC-SpoutL1-Pad15): track 35.6 -> 83.8 mm
- net Net-(MC-LeverL1-Pad16): track 61.3 -> 105.6 mm, vias 2 -> 0
- net Net-(SoundVisionR1-Pad2): track 27.0 -> 69.5 mm
- net Net-(MC-SpoutR1-Pad15): track 81.3 -> 121.4 mm, vias 0 -> 2
- net Net-(HandleL-ToMotor1-Pad1): track 91.4 -> 53.0 mm, vias 0 -> 1
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- removed copper zone on F.Cu, net +5V
Other:
- board size 151.1 x 123.2 mm -> 222.2 x 73.7 mm
