File: pcb/controller/controller.sch (KiCad schematic (older format))
At the start: 35 parts, among them J12V1 Screw_Terminal_01x02, J12V2 Screw_Terminal_01x02, J12V3 Screw_Terminal_01x02, J12V4 Screw_Terminal_01x02, J2 RJ45, J5V1 Screw_Terminal_01x02, J5V2 Screw_Terminal_01x02, J9V1 Screw_Terminal_01x02, SW12 SW12V, SW5 SW5V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

Commit message: Renamed and cleaned up rescue libs so the project is self-contained.
Parts:
- U1: symbol MC_board-rescue:Teensy3.2-teensy -> teensy:Teensy3.2
- U2: symbol MC_board-rescue:MAX98306-spatialsparrow -> spatialsparrow:MAX98306
Changed lines of the file:
@@
 $EndComp
 $Comp
-L MC_board-rescue:MAX98306-spatialsparrow U2
+L spatialsparrow:MAX98306 U2
 U 1 1 5F0C05CB
 P 3850 9750
@@
 $EndComp
 $Comp
-L MC_board-rescue:Teensy3.2-teensy U1
+L teensy:Teensy3.2 U1
 U 1 1 5EFE2FDF
 P 13250 3450

Commit message: Controller pcb working version.
Parts:
- HandleL-ToMotor1, HandleR-ToMotor1, SpoutL-ToMotor1, SpoutR-ToMotor1: footprint teensey:TerminalBlock_TE_282825-4_1x04_P5.08mm_Horizontal -> teensy:TerminalBlock_TE_282825-4_1x04_P5.08mm_Horizontal
- J12V1, J12V2, J12V3, J12V4, J5V1, J5V2, J9V1, distractor1: footprint teensey:TerminalBlock_TE_282825-2_1x02_P5.08mm_Horizontal -> teensy:TerminalBlock_TE_282825-2_1x02_P5.08mm_Horizontal
- J2: footprint teensey:RJ45_sparkfun -> teensy:RJ45_sparkfun
- JP1: footprint Jumper:SolderJumper-2_P1.3mm_Open_Pad1.0x1.5mm -> TestPoint:TestPoint_2Pads_Pitch5.08mm_Drill1.3mm
- SoundVisionL1, SoundVisionR1: footprint teensey:TerminalBlock_TE_282825-6_1x06_P5.08mm_Horizontal -> teensy:TerminalBlock_TE_282825-6_1x06_P5.08mm_Horizontal
- ToHandleL1, ToHandleR1, sync_trigger_out1: footprint teensey:TerminalBlock_TE_282825-5_1x05_P5.08mm_Horizontal -> teensy:TerminalBlock_TE_282825-5_1x05_P5.08mm_Horizontal
- U1: footprint teensey:Teensy30_31_32_LC -> teensy:Teensy30_31_32_LC
Changed lines of the file:
@@
 F 0 "HandleL-ToMotor1" H 6580 2642 50  0000 L CNN
 F 1 "Screw_Terminal_01x04" H 6580 2551 50  0000 L CNN
-F 2 "teensey:TerminalBlock_TE_282825-4_1x04_P5.08mm_Horizontal" H 6500 2650 50  0001 C CNN
+F 2 "teensy:TerminalBlock_TE_282825-4_1x04_P5.08mm_Horizontal" H 6500 2650 50  0001 C CNN
 F 3 "~" H 6500 2650 50  0001 C CNN
 	1    6500 2650
@@
 F 0 "HandleR-ToMotor1" H 6550 4550 50  0000 L CNN
 F 1 "Screw_Terminal_01x04" H 6650 4450 50  0000 L CNN
-F 2 "teensey:TerminalBlock_TE_282825-4_1x04_P5.08mm_Horizontal" H 6550 4300 50  0001 C CNN
+F 2 "teensy:TerminalBlock_TE_282825-4_1x04_P5.08mm_Horizontal" H 6550 4300 50  0001 C CNN
 F 3 "~" H 6550 4300 50  0001 C CNN
 	1    6550 4300
@@
 F 0 "SpoutR-ToMotor1" H 4200 4200 50  0000 L CNN
 F 1 "Screw_Terminal_01x04" H 4150 4100 50  0000 L CNN
-F 2 "teensey:TerminalBlock_TE_282825-4_1x04_P5.08mm_Horizontal" H 4500 4550 50  0001 C CNN
+F 2 "teensy:TerminalBlock_TE_282825-4_1x04_P5.08mm_Horizontal" H 4500 4550 50  0001 C CNN
 F 3 "~" H 4500 4550 50  0001 C CNN
 	1    4500 4550
@@
 F 0 "SpoutL-ToMotor1" H 4250 2300 50  0000 L CNN
 F 1 "Screw_Terminal_01x04" H 4200 2200 50  0000 L CNN
-F 2 "teensey:TerminalBlock_TE_282825-4_1x04_P5.08mm_Horizontal" H 4500 2600 50  0001 C CNN
+F 2 "teensy:TerminalBlock_TE_282825-4_1x04_P5.08mm_Horizontal" H 4500 2600 50  0001 C CNN
 F 3 "~" H 4500 2600 50  0001 C CNN
 	1    4500 2600
@@
 F 0 "ToHandleR1" H 7318 6525 50  0000 C CNN
 F 1 "Screw_Terminal_01x05" H 7318 6616 50  0000 C CNN
-F 2 "teensey:TerminalBlock_TE_282825-5_1x05_P5.08mm_Horizontal" H 7400 6950 50  0001 C CNN
+F 2 "teensy:TerminalBlock_TE_282825-5_1x05_P5.08mm_Horizontal" H 7400 6950 50  0001 C CNN
 F 3 "~" H 7400 6950 50  0001 C CNN
 	1    7400 6950
@@
 F 0 "ToHandleL1" H 10418 6525 50  0000 C CNN
 F 1 "Screw_Terminal_01x05" H 10418 6616 50  0000 C CNN
-F 2 "teensey:TerminalBlock_TE_282825-5_1x05_P5.08mm_Horizontal" H 10500 6950 50  0001 C CNN
+F 2 "teensy:TerminalBlock_TE_282825-5_1x05_P5.08mm_Horizontal" H 10500 6950 50  0001 C CNN
 F 3 "~" H 10500 6950 50  0001 C CNN
 	1    10500 6950
@@
 F 0 "J2" H 2007 9867 50  0000 C CNN
 F 1 "RJ45" H 2007 9776 50  0000 C CNN
-F 2 "teensey:RJ45_sparkfun" V 1950 9225 50  0001 C CNN
+F 2 "teensy:RJ45_sparkfun" V 1950 9225 50  0001 C CNN
 F 3 "~" V 1950 9225 50  0001 C CNN
 	1    1950 9200
@@
 F 0 "U1" H 13250 5087 60  0000 C CNN
 F 1 "Teensy3.2" H 13250 4981 60  0000 C CNN
-F 2 "teensey:Teensy30_31_32_LC" H 13250 2700 60  0001 C CNN
+F 2 "teensy:Teensy30_31_32_LC" H 13250 2700 60  0001 C CNN
 F 3 "" H 13250 2700 60  0000 C CNN
 	1    13250 3450
@@
 F 0 "J12V2" H 5380 12592 50  0000 L CNN
 F 1 "Screw_Terminal_01x02" H 5380 12501 50  0000 L CNN
-F 2 "teensey:TerminalBlock_TE_282825-2_1x02_P5.08mm_Horizontal" H 5300 12600 50  0001 C CNN
+F 2 "teensy:TerminalBlock_TE_282825-2_1x02_P5.08mm_Horizontal" H 5300 12600 50  0001 C CNN
 F 3 "~" H 5300 12600 50  0001 C CNN
 	1    5300 12600
@@
 F 0 "SoundVisionR1" H 5368 6785 50  0000 C CNN
 F 1 "Screw_Terminal_01x06" H 5368 6876 50  0000 C CNN
-F 2 "teensey:TerminalBlock_TE_282825-6_1x06_P5.08mm_Horizontal" H 5450 7250 50  0001 C CNN
+F 2 "teensy:TerminalBlock_TE_282825-6_1x06_P5.08mm_Horizontal" H 5450 7250 50  0001 C CNN
 F 3 "~" H 5450 7250 50  0001 C CNN
 	1    5450 7250
@@
 F 0 "SoundVisionL1" H 3068 6785 50  0000 C CNN
 F 1 "Screw_Terminal_01x06" H 3068 6876 50  0000 C CNN
-F 2 "teensey:TerminalBlock_TE_282825-6_1x06_P5.08mm_Horizontal" H 3150 7250 50  0001 C CNN
+F 2 "teensy:TerminalBlock_TE_282825-6_1x06_P5.08mm_Horizontal" H 3150 7250 50  0001 C CNN
 F 3 "~" H 3150 7250 50  0001 C CNN
 	1    3150 7250
@@
 F 0 "sync_trigger_out1" H 8168 2525 50  0000 C CNN
 F 1 "Screw_Terminal_01x05" H 8168 2616 50  0000 C CNN
-F 2 "teensey:TerminalBlock_TE_282825-5_1x05_P5.08mm_Horizontal" H 8250 2950 50  0001 C CNN
+F 2 "teensy:TerminalBlock_TE_282825-5_1x05_P5.08mm_Horizontal" H 8250 2950 50  0001 C CNN
 F 3 "~" H 8250 2950 50  0001 C CNN
 	1    8250 2950
@@
 F 0 "J12V3" H 5380 12892 50  0000 L CNN
 F 1 "Screw_Terminal_01x02" H 5380 12801 50  0000 L CNN
-F 2 "teensey:TerminalBlock_TE_282825-2_1x02_P5.08mm_Horizontal" H 5300 12900 50  0001 C CNN
+F 2 "teensy:TerminalBlock_TE_282825-2_1x02_P5.08mm_Horizontal" H 5300 12900 50  0001 C CNN
 F 3 "~" H 5300 12900 50  0001 C CNN
 	1    5300 12900
@@
 F 0 "J12V4" H 5380 13192 50  0000 L CNN
 F 1 "Screw_Terminal_01x02" H 5380 13101 50  0000 L CNN
-F 2 "teensey:TerminalBlock_TE_282825-2_1x02_P5.08mm_Horizontal" H 5300 13200 50  0001 C CNN
+F 2 "teensy:TerminalBlock_TE_282825-2_1x02_P5.08mm_Horizontal" H 5300 13200 50  0001 C CNN
 F 3 "~" H 5300 13200 50  0001 C CNN
 	1    5300 13200
@@
 F 0 "J5V1" H 5380 13692 50  0000 L CNN
 F 1 "Screw_Terminal_01x02" H 5380 13601 50  0000 L CNN
-F 2 "teensey:TerminalBlock_TE_282825-2_1x02_P5.08mm_Horizontal" H 5300 13700 50  0001 C CNN
+F 2 "teensy:TerminalBlock_TE_282825-2_1x02_P5.08mm_Horizontal" H 5300 13700 50  0001 C CNN
 F 3 "~" H 5300 13700 50  0001 C CNN
 	1    5300 13700
@@
 F 0 "J5V2" H 5380 14042 50  0000 L CNN
 F 1 "Screw_Terminal_01x02" H 5380 13951 50  0000 L CNN
-F 2 "teensey:TerminalBlock_TE_282825-2_1x02_P5.08mm_Horizontal" H 5300 14050 50  0001 C CNN
+F 2 "teensy:TerminalBlock_TE_282825-2_1x02_P5.08mm_Horizontal" H 5300 14050 50  0001 C CNN
 F 3 "~" H 5300 14050 50  0001 C CNN
 	1    5300 14050
@@
 F 0 "J12V1" H 5380 12292 50  0000 L CNN
 F 1 "Screw_Terminal_01x02" H 5380 12201 50  0000 L CNN
-F 2 "teensey:TerminalBlock_TE_282825-2_1x02_P5.08mm_Horizontal" H 5300 12300 50  0001 C CNN
+F 2 "teensy:TerminalBlock_TE_282825-2_1x02_P5.08mm_Horizontal" H 5300 12300 50  0001 C CNN
 F 3 "~" H 5300 12300 50  0001 C CNN
 	1    5300 12300
@@
 F 0 "J9V1" H 5380 14542 50  0000 L CNN
 F 1 "Screw_Terminal_01x02" H 5380 14451 50  0000 L CNN
-F 2 "teensey:TerminalBlock_TE_282825-2_1x02_P5.08mm_Horizontal" H 5300 14550 50  0001 C CNN
+F 2 "teensy:TerminalBlock_TE_282825-2_1x02_P5.08mm_Horizontal" H 5300 14550 50  0001 C CNN
 F 3 "~" H 5300 14550 50  0001 C CNN
 	1    5300 14550
@@
 F 0 "distractor1" H 3980 8592 50  0000 L CNN
 F 1 "Screw_Terminal_01x02" H 3980 8501 50  0000 L CNN
-F 2 "teensey:TerminalBlock_TE_282825-2_1x02_P5.08mm_Horizontal" H 3900 8600 50  0001 C CNN
+F 2 "teensy:TerminalBlock_TE_282825-2_1x02_P5.08mm_Horizontal" H 3900 8600 50  0001 C CNN
 F 3 "~" H 3900 8600 50  0001 C CNN
 	1    3900 8600
@@
 F 0 "JP1" H 3550 13985 50  0000 C CNN
 F 1 "gnd jumper" H 3550 13894 50  0000 C CNN
-F 2 "Jumper:SolderJumper-2_P1.3mm_Open_Pad1.0x1.5mm" H 3550 13750 50  0001 C CNN
+F 2 "TestPoint:TestPoint_2Pads_Pitch5.08mm_Drill1.3mm" H 3550 13750 50  0001 C CNN
 F 3 "~" H 3550 13750 50  0001 C CNN
 	1    3550 13750
